File: rev1/a_duck.kicad_pcb (KiCad board)
At the start: 2 copper layers, 135.1 x 107.9 mm, 38 parts

Commit message: Added V1 of PCB with routing
Routing:
- net P9: track 38.2 -> 199.3 mm, vias 0 -> 3
- net P8: track 35.1 -> 192.1 mm, vias 0 -> 3
- net P7: track 81.3 -> 232.9 mm, vias 0 -> 4
- net P6: track 91.3 -> 224.0 mm, vias 0 -> 4
- net P5: track 94.7 -> 216.8 mm, vias 0 -> 4
- net P15: track 129.8 -> 169.5 mm
- net P14: track 121.9 -> 147.7 mm
- net VCC: track 5.35 -> 30.9 mm
- net P10: track 55.2 -> 76.6 mm, vias 3 -> 4
- net GND: track 9.46 -> 28.6 mm
- net P16: track 118.3 -> 130.2 mm
